File: v1.2/DIB_interface.kicad_sch (KiCad schematic)
At the start: 16 parts, among them IC1 M24C32-WMN6P, IC2 SI8641NSOIC-16, IC3 SI8641NSOIC-16, J1 4907

Commit message: BOM update
Parts:
- added X2: ZL263-20DG, PCM_EEZ_connectors:SSW-110-02-T-D-RA, symbol PCM_EEZ_connectors:Conn_2Rows-20Pins
- added X4, X5: 87833-1032, PCM_EEZ_connectors:DS1014-10RF1B, symbol Connector_Generic:Conn_02x05_Odd_Even
- IC2, IC3: value SI8641NSOIC-16 -> SI8641BB-B-IS1
- X3: renamed from X1; value ~ -> 77317-104-28LF
- renumbered J1 to X1
Connections:
- net GND: now also X4.1 (Pin_1), X4.10 (Pin_10), X4.2 (Pin_2), X4.5 (Pin_5), X4.6 (Pin_6), X5.1 (Pin_1), X5.10 (Pin_10), X5.2 (Pin_2), X5.5 (Pin_5), X5.6 (Pin_6)
- new net ADIB1_ID0: X4.7 (Pin_7)
- new net ADIB1_ID1: X4.9 (Pin_9)
- new net ADIB1_ID2: X4.8 (Pin_8)
- new net ADIB2_ID0: X5.7 (Pin_7)
- new net ADIB2_ID1: X5.9 (Pin_9)
- new net ADIB2_ID2: X5.8 (Pin_8)
- new net AFE1N: X4.3 (Pin_3)
- new net AFE1P: X4.4 (Pin_4)
- new net AFE2N: X5.3 (Pin_3)
- new net AFE2P: X5.4 (Pin_4)
Other:
- note added: "+3V3 1 NFAULT 3 DIB_SCL 5 Gnd 7 DIB_CSA 9 Gnd 9 DIB_SCLK 13 DIB_MOSI 15 DIB_A0 17 DIB_A1 19 +12V 21 +5V 23 Gnd 25 UART_TX 27"
- note added: "10-pin ADIB socket"
- note added: "2 +Vaux 4 ~{RESET} 6 OE_SYNC 8 DIB_SDA 10 DIB_IRQ 12 DIB_CSB 14 DIB_MISO 16 Gnd 18 DIB_A2 20 Gnd 22 +12V 24 +5V 26 Gnd 28 UART_RX"
- note added: "2 Guard+ 4 AIN+ 6 Guard+ 8 ADIB_ID2 10 ID_Gnd"
- note added: "2 OUTC+ 4 OUTC+ 6 OUTC+ 8 POST_OUT+ 10 POST_OUT+ 12 POST_OUT- 14 POST_OUT- 16 OUTC- 18 OUTC- 20 OUTC-"
- note added: "20-pin power socket"
- note added: "ADIB connectors (optional)"
- note added: "DIB host connector (mandatory)"
- note added: "DIB power connector (optional)"
- note added: "Guard- 1 AIN- 3 Guard- 5 ADIB_ID0 7 ADIB_ID1 9"
- note added: "OUTC+ 1 OUTC+ 3 OUTC+ 5 POST_OUT+ 7 POST_OUT+ 9 POST_OUT- 11 POST_OUT- 13 POST_OUT -15 OUTC- 17 OUTC- 19"
- note removed: "+12V 21"
- note removed: "+3V3 1"
- note removed: "+5V 23"
- note removed: "10 DIB_IRQ"
- note removed: "12 DIB_CSB"
- note removed: "14 DIB_MISO"
- note removed: "16 Gnd"
- note removed: "18 DIB_A2"
- note removed: "2 +Vaux"
- note removed: "20 Gnd"
- note removed: "22 +12V"
- note removed: "24 +5V"
- note removed: "26 BOOT"
- note removed: "28 UART_TX"
- note removed: "4 NRESET"
- note removed: "6 OE_SYNC"
- note removed: "8 DIB_SDA"
- note removed: "DIB connector"
- note removed: "DIB_A0 17"
- note removed: "DIB_A1 19"
- note removed: "DIB_CSA 9"
- note removed: "DIB_MOSI 15"
- note removed: "DIB_SCL 5"
- note removed: "DIB_SCLK 13"
- note removed: "Gnd 11"
- note removed: "Gnd 25"
- note removed: "Gnd 7"
- note removed: "NFAULT 3"
- note removed: "UART_RX 27"
