File: v1.2/EEZ DIB 1.2 template.kicad_pcb (KiCad board)
At the start: 4 copper layers, 146 x 95 mm, 28 parts, among them IC1 M24C32-WMN6P, IC2 SI8641NSOIC-16, IC3 SI8641NSOIC-16, J1 4907, X2 87833-1032, X3 87833-1032

Commit message: BOM update
Parts:
- removed the X2 at (120.5, 65.5)
- added X1: ZL263-20DG, PCM_EEZ_connectors:SSW-110-02-T-D-RA, F.Cu at (116.0, 140.0)
- added X4: 87833-1032, PCM_EEZ_connectors:DS1014-10RF1B, F.Cu at (140.5, 65.5)
- IC2, IC3: value SI8641NSOIC-16 -> SI8641BB-B-IS1
- X2: renamed from X1; value ~ -> 77317-104-28LF
- moved LOGO1 123.7 mm to (191.1, 62.8)
- moved LOGO2 123.7 mm to (200.2, 64.2)
- moved LOGO3 123.7 mm to (206.4, 63.9)
- moved LOGO4 123.7 mm to (213.0, 64.3)
- moved X3 20.0 mm to (120.5, 65.5)
Connections:
- net /ADIB connectors (optional)/AFE2N renamed /DIB v1.2 interface/AFE1N
- net /ADIB connectors (optional)/AFE2P renamed /DIB v1.2 interface/AFE1P
- X3 pad 7: ADIB2_ID0 -> ADIB1_ID0
- X3 pad 8: ADIB2_ID2 -> ADIB1_ID2
- X3 pad 9: ADIB2_ID1 -> ADIB1_ID1

Commit message: 3D model updated
Parts:
- added FM5: ~, PCM_EEZ_unsorted:DIB module front mask, F.Cu at (75.0, 161.0)
- renumbered J1 to X1, X1 to X2, X2 to X3, X3 to X4, X4 to X5
