File: v1.2/EEZ DIB 1.2 template.kicad_sch (KiCad schematic)
At the start: 10 parts

Commit message: BOM update
Other:
- removed sheet ADIB connectors (optional)
Changed lines of the file:
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@@
-	)
-	(sheet
-		(at 60.96 30.48)
-		(size 12.7 3.81)
-		(fields_autoplaced yes)
-		(stroke
-			(width 0)
-			(type solid)
-		)
-		(fill
-			(color 0 0 0 0.0000)
-		)
-		(property "Sheetname" "ADIB connectors (optional)"
-			(at 60.96 29.7684 0)
-			(effects
-				(font
-					(size 1.27 1.27)
-				)
-				(justify left bottom)
-			)
-		)
-		(property "Sheetfile" "ADIB.kicad_sch"
-			(at 60.96 34.8746 0)
-			(effects
-				(font
-					(size 1.27 1.27)
-				)
-				(justify left top)
-				(hide yes)
-			)
-		)
-		(instances
-			(project "EEZ DIB 1.2 template"
-				(path "/8165d74e-be16-4c9d-8240-91910dc4b43e"
-					(page "6")
-				)
-			)
-		)
 	)
 	(sheet

Commit message: 3D model updated
Parts:
- added FM5: ~, PCM_EEZ_unsorted:DIB module front mask, symbol PCM_EEZ_unsorted:DIB module front mask
Other:
- note added: "Front mask"
Changed lines of the file:
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@@
 	(title_block
 		(title "${project_name}")
-		(date "2024-12-15")
+		(date "2025-02-06")
 		(rev "${project_version}")
 		(company "${project_creator}")
@@
 		(pts
 			(xy 119.38 177.8) (xy 15.24 177.8)
+		)
+		(stroke
+			(width 0.1524)
+			(type dash)
+			(color 194 194 194 1)
+		)
+	)
+	(polyline
+		(pts
+			(xy 119.38 177.8) (xy 144.78 177.8)
+		)
+		(stroke
+			(width 0.1524)
+			(type dash)
+			(color 194 194 194 1)
+		)
+	)
+	(polyline
+		(pts
+			(xy 144.78 177.8) (xy 144.78 195.58)
 		)
 		(stroke
@@
 		)
 	)
+	(text "Front mask"
+		(exclude_from_sim no)
+		(at 121.92 182.88 0)
+		(effects
+			(font
+				(size 1.778 1.5113)
+				(color 194 194 194 1)
+			)
+			(justify left bottom)
+		)
+	)
 	(symbol
 		(lib_id "PCM_EEZ_symbols:FIDUCIAL")
@@
 					(unit 1)
 				)
+			)
+		)
+	)
+	(symbol
+		(lib_id "PCM_EEZ_unsorted:DIB module front mask")
+		(at 128.905 184.15 0)
+		(unit 1)
+		(exclude_from_sim no)
+		(in_bom yes)
+		(on_board yes)
+		(dnp no)
+		(fields_autoplaced yes)
+		(property "Reference" "FM5"
+			(at 133.985 187.0074 0)
+			(effects
+				(font
+					(size 1.27 1.27)
+				)
+				(justify left)
+			)
+		)
+		(property "Value" "~"
+			(at 133.985 188.9125 0)
+			(effects
+				(font
+					(size 1.27 1.27)
+				)
+				(justify left)
+			)
+		)
+		(property "Footprint" "PCM_EEZ_unsorted:DIB module front mask"
+			(at 128.905 184.15 0)
+			(effects
+				(font
+					(size 1.27 1.27)
+				)
+				(hide yes)
+			)
+		)
+		(property "Datasheet" ""
+			(at 128.905 184.15 0)
+			(effects
+				(font
+					(size 1.27 1.27)
+				)
+				(hide yes)
+			)
+		)
+		(property "Description" ""
+			(at 128.905 184.15 0)
+			(effects
+				(font
+					(size 1.27 1.27)
+				)
+				(hide yes)
+			)
+		)
+		(instances
+			(project ""
+				(path "/8165d74e-be16-4c9d-8240-91910dc4b43e"
+					(reference "FM5")
+					(unit 1)
+				)
